Commit message: add the urddf description

File: src/arduinobot_description/urdf/arduinobot.urdf.xacro (robot description, xacro)
@@ -1,38 +1,115 @@
-<?xml version="1.0"?>
-<robot xmlns:xacro="http://www.ros.org/wiki/xacro" name="arduinobot">
-    <!-- Useful Variables (Properties) -->
-    <xacro:property name="PI" value="3.14159265359" />
-    <xacro:property name="effort" value="30" />
-    <xacro:property name="velocity" value="10" />
-    <!-- Links -->
-    <link name="world"/>
-    <link name="base_link">
+<?xml version= "1.0"?>
+<robot xmlns:xacro="https://www.ros.org/wiki/xacro" name="arduinobot">
+<xacro:property name="PI" value = "3.14159265359"/>
+<xacro:property name ="effort" value = "30"/>
+<xacro:property name="velocity" value = "10"/>
+    <link name = "world"/>
+    <link name = "base_link">
         <visual>
-            <origin rpy="0 0 0" xyz="-0.5 -0.5 0"/>
+            <origin rpy = "0 0 0" xyz = "-0.5 -0.5 0"/>
             <geometry>
-                <mesh filename="package://arduinobot_description/mesh/basement.STL" scale="0.01 0.01 0.01"/>
+                <mesh filename="package://arduinobot_description/mesh/basement.STL" scale = "0.01 0.01 0.01" />
             </geometry>
         </visual>
     </link>
-    <link name="base_plate">
+    <link name = "base_plate">
         <visual>
-            <origin rpy="0 0 0" xyz="-0.39 -0.39 -0.56"/>
+            <origin rpy = "0 0 0" xyz = "-0.39 -0.39 -0.56"/>
             <geometry>
-                <mesh filename="package://arduinobot_description/mesh/base_plate.STL" scale="0.01 0.01 0.01"/>
+                <mesh filename="package://arduinobot_description/mesh/base_plate.STL" scale = "0.01 0.01 0.01" />
             </geometry>
         </visual>
     </link>
-    <!-- Joints -->
-    <joint name="virtual_joint" type="fixed">
-        <parent link="world"/>
-        <child link="base_link"/>
-        <origin xyz="0 0 0" rpy="0 0 0"/>
+    <link name="forward_drive_arm">
+        <visual>
+            <origin rpy=" 0 -${PI/2} ${PI/2}" xyz="0.19 0.06 -0.08"/>
+            <geometry>
+                <mesh filename="package://arduinobot_description/mesh/forward_drive_arm.STL" scale="0.01 0.01 0.01"/>
+            </geometry>
+        </visual>
+    </link>
+    <link name="horizontal_arm">
+        <visual>
+            <origin rpy="${PI/2} 0 ${PI/2}" xyz="-0.03 -0.4 -0.06"/>
+            <geometry>
+                <mesh filename="package://arduinobot_description/mesh/horizontal_arm.STL" scale="0.01 0.01 0.01"/>
+            </geometry>
+        </visual>
+    </link>
+    <link name="claw_support">
+        <visual>
+            <origin rpy="0 0 ${PI/2}" xyz="0 -0.05 -0.15"/>
+            <geometry>
+                <mesh filename="package://arduinobot_description/mesh/claw_support.STL" scale="0.01 0.01 0.01"/>
+            </geometry>
+        </visual>
+    </link>
+    <link name="gripper_right">
+        <visual>
+            <origin rpy="0 0 -${PI/2}" xyz="-0.1 0.50 -0.1"/>
+            <geometry>
+                <mesh filename="package://arduinobot_description/mesh/right_finger.STL" scale="0.01 0.01 0.01"/>
+            </geometry>
+        </visual>
+    </link>
+    <link name="gripper_left">
+        <visual>
+            <origin rpy="0 0 -${PI/2}" xyz="-0.04 0.50 -0.1"/>
+            <geometry>
+                <mesh filename="package://arduinobot_description/mesh/left_finger.STL" scale="0.01 0.01 0.01"/>
+            </geometry>
+        </visual>
+    </link>
+    <link name="tool_link"></link>
+    <joint name  = "virtual_joint" type ="fixed" >
+        <parent link = "world"/>
+        <child link =  "base_link"/>
+        <origin rpy= "0 0 0" xyz = "0 0 0"/>
     </joint>
-    <joint name ="joint_1" type="revolute">
-        <parent link="base_link"/>
-        <child link = "base_plate"/>
-        <origin xyz="0 0 0.307"/>
-        <axis xyz="0 0 1"/>
+    <joint name  = "joint_1" type ="revolute">
+        <parent link = "base_link"/>
+        <child link =  "base_plate"/>
+        <origin xyz = "0 0 0.307"/>
+        <axis xyz= "0 0 1"/>
+        <limit lower= "-${PI/2}" upper= "${PI/2}" effort= "${effort}" velocity="${velocity}"/>
+    </joint>
+    <joint name ="joint_2" type="revolute">
+        <parent link="base_plate"/>
+        <child link = "forward_drive_arm"/>
+        <origin xyz="-0.02 0 0.35"/>
+        <axis xyz="1 0 0"/>
         <limit lower="-${PI/2}" upper="${PI/2}" effort="${effort}" velocity="${velocity}"/>
     </joint>
+    <joint name ="joint_3" type="revolute">
+        <parent link="forward_drive_arm"/>
+        <child link = "horizontal_arm"/>
+        <origin xyz="0 0 0.8"/>
+        <axis xyz="1 0 0"/>
+        <limit lower="-${PI/2}" upper="${PI/2}" effort="${effort}" velocity="${velocity}"/>
+    </joint>
+    <joint name ="horizontal_arm_to_claw_support" type="fixed">
+        <parent link="horizontal_arm"/>
+        <child link = "claw_support"/>
+        <origin xyz="0 0.82 0"/>
+    </joint>
+    <joint name ="joint_4" type="revolute">
+        <parent link="claw_support"/>
+        <child link = "gripper_right"/>
+        <origin xyz="-0.04 0.13 -0.1"/>
+        <axis xyz="0 0 1"/>
+        <limit lower="-${PI/2}" upper="0" effort="${effort}" velocity="${velocity}"/>
+    </joint>
+    <joint name ="joint_5" type="revolute">
+        <parent link="claw_support"/>
+        <child link = "gripper_left"/>
+        <origin xyz="-0.22 0.13 -0.1"/>
+        <axis xyz="0 0 1"/>
+        <limit lower="0" upper="${PI/2}" effort="${effort}" velocity="${velocity}"/>
+        <mimic joint="joint_4" multiplier="-1" offset="0"/>
+    </joint>
+    <joint name ="gripper_right_to_tool" type="fixed">
+        <parent link="gripper_right"/>
+        <child link = "tool_link"/>
+        <origin xyz="0 0 0"/>
+    </joint>
 </robot>

Commit message: add rviz file,gazebo launch files and make the gazebo plugin

File: src/arduinobot_description/urdf/arduinobot.urdf.xacro (robot description, xacro)
@@ -1,17 +1,43 @@
 <?xml version= "1.0"?>
 <robot xmlns:xacro="https://www.ros.org/wiki/xacro" name="arduinobot">
-<xacro:property name="PI" value = "3.14159265359"/>
-<xacro:property name ="effort" value = "30"/>
-<xacro:property name="velocity" value = "10"/>
+    <xacro:property name="PI" value = "3.14159265359"/>
+    <xacro:property name="effort" value = "30"/>
+    <xacro:property name="velocity" value = "10"/>
+    <xacro:macro name="default_inirtial" params="mass">
+        <inertial>
+            <mass value="${mass}"/>
+            <inertia ixx="1" ixy="0.0" ixz="0.0" iyy="1" iyz="0.0" izz="1"/>
+        </inertial>
+    </xacro:macro>
+    <xacro:macro name="default_transmission" params="number">
+        <transmission name="transmission_${number}">
+            <type>transmission_interface/SimpleTransmission</type>
+            <joint name="joint${number}">
+                <hardwareInterface>hardware_interface/PositionJointInterface</hardwareInterface>
+            </joint>
+            <actuator name="motor_${number}">
+                <mechanicalReduction>1.0</mechanicalReduction>
+                <hardwareInterface>hardware_interface/PositionJointInterface</hardwareInterface>
+            </actuator>
+        </transmission>
+    </xacro:macro>
     <link name = "world"/>
     <link name = "base_link">
+    <xacro:default_inirtial mass="1.0"/>
         <visual>
             <origin rpy = "0 0 0" xyz = "-0.5 -0.5 0"/>
             <geometry>
-                <mesh filename="package://arduinobot_description/mesh/basement.STL" scale = "0.01 0.01 0.01" />
-            </geometry>
-        </visual>
+                 <mesh filename="package://arduinobot_description/mesh/basement.STL" scale = "0.01 0.01 0.01" />
+            </geometry>
+        </visual>
+        <collision>
+            <origin rpy = "0 0 0" xyz = "-0.5 -0.5 0"/>
+            <geometry>
+                  <mesh filename="package://arduinobot_description/mesh/basement.STL" scale = "0.01 0.01 0.01" />
+            </geometry>
+        </collision>
     </link>
     <link name = "base_plate">
+    <xacro:default_inirtial mass="0.1"/>
         <visual>
             <origin rpy = "0 0 0" xyz = "-0.39 -0.39 -0.56"/>
@@ -20,6 +46,13 @@
             </geometry>
         </visual>
+        <collision>
+            <origin rpy = "0 0 0" xyz = "-0.39 -0.39 -0.56"/>
+            <geometry>
+                  <mesh filename="package://arduinobot_description/mesh/base_plate.STL" scale = "0.01 0.01 0.01" />
+            </geometry>
+        </collision>
     </link>
     <link name="forward_drive_arm">
+    <xacro:default_inirtial mass="0.1"/>
         <visual>
             <origin rpy=" 0 -${PI/2} ${PI/2}" xyz="0.19 0.06 -0.08"/>
@@ -28,6 +61,13 @@
             </geometry>
         </visual>
+        <collision>
+            <origin rpy=" 0 -${PI/2} ${PI/2}" xyz="0.19 0.06 -0.08"/>
+            <geometry>
+                <mesh filename="package://arduinobot_description/mesh/forward_drive_arm.STL" scale="0.01 0.01 0.01"/>
+            </geometry>
+        </collision>
     </link>
     <link name="horizontal_arm">
+    <xacro:default_inirtial mass="0.1"/>
         <visual>
             <origin rpy="${PI/2} 0 ${PI/2}" xyz="-0.03 -0.4 -0.06"/>
@@ -36,6 +76,13 @@
             </geometry>
         </visual>
+        <collision>
+            <origin rpy="${PI/2} 0 ${PI/2}" xyz="-0.03 -0.4 -0.06"/>
+            <geometry>
+                <mesh filename="package://arduinobot_description/mesh/horizontal_arm.STL" scale="0.01 0.01 0.01"/>
+            </geometry>
+        </collision>
     </link>
     <link name="claw_support">
+    <xacro:default_inirtial mass="0.05"/>
         <visual>
             <origin rpy="0 0 ${PI/2}" xyz="0 -0.05 -0.15"/>
@@ -44,6 +91,13 @@
             </geometry>
         </visual>
+        <collision>
+             <origin rpy="0 0 ${PI/2}" xyz="0 -0.05 -0.15"/>
+             <geometry>
+                <mesh filename="package://arduinobot_description/mesh/claw_support.STL" scale="0.01 0.01 0.01"/>
+            </geometry>
+        </collision>
     </link>
     <link name="gripper_right">
+    <xacro:default_inirtial mass="0.01"/>
         <visual>
             <origin rpy="0 0 -${PI/2}" xyz="-0.1 0.50 -0.1"/>
@@ -52,6 +106,13 @@
             </geometry>
         </visual>
+        <collision>
+            <origin rpy="0 0 -${PI/2}" xyz="-0.1 0.50 -0.1"/>
+            <geometry>
+                <mesh filename="package://arduinobot_description/mesh/right_finger.STL" scale="0.01 0.01 0.01"/>
+            </geometry>
+        </collision>
     </link>
     <link name="gripper_left">
+    <xacro:default_inirtial mass="0.01"/>
         <visual>
             <origin rpy="0 0 -${PI/2}" xyz="-0.04 0.50 -0.1"/>
@@ -60,4 +121,10 @@
             </geometry>
         </visual>
+        <collision>
+             <origin rpy="0 0 -${PI/2}" xyz="-0.04 0.50 -0.1"/>
+            <geometry>
+                <mesh filename="package://arduinobot_description/mesh/left_finger.STL" scale="0.01 0.01 0.01"/>
+            </geometry>
+        </collision>
     </link>
     <link name="tool_link"></link>
@@ -113,3 +180,22 @@
         <origin xyz="0 0 0"/>
     </joint>
+    <xacro:default_transmission number="1"/>
+    <xacro:default_transmission number="2"/>
+    <xacro:default_transmission number="3"/>
+    <xacro:default_transmission number="4"/>
+    <gazebo>
+        <plugin name="gazebo_ros_control" filename="libgazebo_ros_control.so">
+            <robotNamespace>/arduinobot</robotNamespace>
+            <robotSimType>gazebo_ros_control/DefaultRobotHWSim</robotSimType>
+            <legacyModeNS>true</legacyModeNS>
+        </plugin>
+        <plugin name="joint_5_mimic_joint_4" filename="libroboticsgroup_upatras_gazebo_mimic_joint_plugin.so">
+            <joint>joint_4</joint>
+            <mimicJoint>joint_5</mimicJoint>
+            <multiplier>-1.0</multiplier>
+            <offset>0</offset>
+            <maxEffort>${effort}</maxEffort>
+            <robotNamespace>/arduinobot</robotNamespace>
+        </plugin>
+    </gazebo>
 </robot>
